Commit message: Added contact sensors to dogBot

File: dogbot_description/urdf/dogbot.xacro (robot description, xacro)
@@ -305,4 +305,15 @@
       <kp value="${kp}" />
       <kd value="${kd}" />
+      <!-- Contact Sensor -->
+      <sensor name="${prefix}_${suffix}_contactsensor_sensor" type="contact">
+        <always_on>true</always_on>
+        <contact>
+          <collision>${prefix}_${suffix}_lowerleg_fixed_joint_lump__${prefix}_${suffix}_foot_collision_5</collision>
+        </contact>
+        <plugin name="${prefix}_${suffix}_foot_plugin" filename="libgazebo_ros_bumper.so">
+          <bumperTopicName>${prefix}_${suffix}_contactsensor_state</bumperTopicName>
+          <frameName>${prefix}_${suffix}_foot</frameName>
+        </plugin>
+      </sensor>
     </gazebo>
     <transmission name="${prefix}_${suffix}_roll_transmition" >
